Commit message: 実環境用のカメラノードの追加

File: src/melodic/myrobot_description/urdf/myrobot.urdf.xacro (robot description, xacro)
@@ -1,4 +1,5 @@
 <?xml version="1.0" encoding="UTF-8"?>
 <robot name="myrobot" xmlns:xacro="http://wiki.ros.org/xacro">
+    <xacro:property name="robot_name" value="myrobot" />
     <gazebo>
         <plugin filename="libgazebo_ros_control.so" name="gazebo_ros_control">
@@ -138,8 +139,8 @@
         <!-- <xacro:f_joint name="${prefix}_camera_base_joint" xyz="${xyz}" parent="${prefix}_J6" child="${prefix}_camera_base" />
         <link name="${prefix}_camera_base" /> -->
-        <xacro:sensor_d435 name="${prefix}_camera" topics_ns="${prefix}_camera" parent="${parent}" publish_pointcloud="0">
+        <xacro:sensor_d435 name="${prefix}_camera" topics_ns="/${robot_name}/${prefix}_camera" parent="${parent}" publish_pointcloud="0">
             <origin xyz="${xyz}" rpy="${rpy}" />
         </xacro:sensor_d435>
-        <xacro:gazebo_d435_override name="${prefix}_camera" topics_ns="${prefix}_camera" publish_pointcloud="1" />
+        <xacro:gazebo_d435_override name="${prefix}_camera" topics_ns="/${robot_name}/${prefix}_camera" publish_pointcloud="1" />
     </xacro:macro>
     <!-- //////////////////////////////////////////////////////////////////////////////////////////////////////////////////////////////////////////////////////////////// -->

Commit message: move common macro to utils.xacro

File: src/melodic/myrobot_description/urdf/myrobot.urdf.xacro (robot description, xacro)
@@ -13,100 +13,5 @@
     <xacro:include filename="$(find realsense2_description)/urdf/_d435.urdf.xacro" />
     <xacro:include filename="$(find myrobot_description)/urdf/gazebo_d435_override.xacro" />
-    <!-- colors definition -->
-    <material name="red">
-        <!-- for revolute -->
-        <color rgba="1.0 0.5 0.5 2.0" />
-    </material>
-    <material name="green">
-        <!-- for prismatic -->
-        <color rgba="0.5 1.0 0.5 2.0" />
-    </material>
-    <material name="blue">
-        <color rgba="0.5 0.5 1.0 2.0" />
-    </material>
-    <material name="white">
-        <color rgba="1.0 1.0 1.0 2.0" />
-    </material>
-    <!-- name=joint is alreadey used in other files? -->
-    <xacro:macro name="f_joint" params="name parent child xyz:='0 0 0' rpy:='0 0 0'">
-        <joint name="${name}" type="fixed">
-            <origin xyz="${xyz}" rpy="${rpy}" />
-            <parent link="${parent}" />
-            <child link="${child}" />
-        </joint>
-    </xacro:macro>
-    <xacro:macro name="_gazebo_joint" params="joint trans reduction:=1">
-        <transmission name="${joint}_trans">
-            <type>transmission_interface/SimpleTransmission</type>
-            <joint name="${joint}">
-                <hardwareInterface>hardware_interface/${trans}</hardwareInterface>
-            </joint>
-            <actuator name="${joint}_motor">
-                <hardwareInterface>hardware_interface/${trans}</hardwareInterface>
-                <mechanicalReduction>${reduction}</mechanicalReduction>
-            </actuator>
-        </transmission>
-    </xacro:macro>
-    <xacro:macro name="a_joint" params="name parent child type axis xyz:='0 0 0' rpy:='0 0 0' eff:=500 low:=-2.967 up:=2.967 vel:=1 damp:=0 fric:=0 trans:=PositionJointInterface">
-        <joint name="${name}" type="${type}">
-            <origin xyz="${xyz}" rpy="${rpy}" />
-            <parent link="${parent}" />
-            <child link="${child}" />
-            <axis xyz="${axis}" />
-            <limit effort="${eff}" lower="${low}" upper="${up}" velocity="${vel}" />
-            <dynamics damping="${damp}" friction="${fric}" />
-        </joint>
-        <xacro:_gazebo_joint joint="${name}" trans="${trans}" />
-    </xacro:macro>
-    <xacro:macro name="_box" params="xyz:='0 0 0' rpy:='0 0 0' size:='0.1 0.1 0.1' mass:=1 color=white">
-        <visual>
-            <origin rpy="${rpy}" xyz="${xyz}" />
-            <geometry>
-                <box size="${size}" />
-            </geometry>
-            <material name="${color}" />
-        </visual>
-        <collision>
-            <origin rpy="${rpy}" xyz="${xyz}" />
-            <geometry>
-                <box size="${size}" />
-            </geometry>
-        </collision>
-        <inertial>
-            <mass value="${mass}" />
-            <origin rpy="${rpy}" xyz="${xyz}" />
-            <inertia ixx="1" ixy="0" ixz="0" iyy="1" iyz="0" izz="1" />
-        </inertial>
-    </xacro:macro>
-    <xacro:macro name="_cylinder" params="xyz:='0 0 0' rpy:='0 0 0' radius:=0.1 length=0.1  mass:=1 color=white">
-        <visual>
-            <origin rpy="${rpy}" xyz="${xyz}" />
-            <geometry>
-                <cylinder radius="${radius}" length="${length}" />
-            </geometry>
-            <material name="${color}" />
-        </visual>
-        <collision>
-            <origin rpy="${rpy}" xyz="${xyz}" />
-            <geometry>
-                <cylinder radius="${radius}" length="${length}" />
-            </geometry>
-        </collision>
-        <inertial>
-            <mass value="${mass}" />
-            <origin rpy="${rpy}" xyz="${xyz}" />
-            <inertia ixx="1" ixy="0" ixz="0" iyy="1" iyz="0" izz="1" />
-        </inertial>
-    </xacro:macro>
-    <xacro:macro name="box_link" params="name xyz:='0 0 0' rpy:='0 0 0' size:='0.1 0.1 0.1' mass:=1 color=white">
-        <link name="${name}">
-            <xacro:_box xyz="${xyz}" rpy="${rpy}" size="${size}" mass="${mass}" color="${color}" />
-        </link>
-    </xacro:macro>
-    <xacro:macro name="cylinder_link" params="name xyz:='0 0 0' rpy:='0 0 0' radius:=0.1 length:=0.1 mass:=1 color=white">
-        <link name="${name}">
-            <xacro:_box xyz="${xyz}" rpy="${rpy}" radius="${radius}" length="${length}" mass="${mass}" color="${color}" />
-        </link>
-    </xacro:macro>
+    <xacro:include filename="$(find myrobot_description)/urdf/utils.xacro" />
     <xacro:macro name="sholder" params="prefix parent xyz l_xyz rpy size up low">
         <xacro:a_joint name="${prefix}_joint_sholder" type="revolute" axis="0 0 1" parent="${parent}" child="${prefix}_sholder" xyz="${xyz}" rpy="${rpy}" up="${up}" low="${low}" />

Commit message: rename base link

File: src/melodic/myrobot_description/urdf/myrobot.urdf.xacro (robot description, xacro)
@@ -73,8 +73,8 @@
     <xacro:property name="sholder_sz" value="0.24" />
     <!-- //////////////////////////////////////////////////////////////////////////////////////////////////////////////////////////////////////////////////////////////// -->
-    <link name="world" />
+    <link name="base_link" />
     <!-- cart -->
     <xacro:box_link name="cart" size="${cart_sx} ${cart_sy} ${cart_sz}" />
-    <xacro:f_joint name="joint_cart" xyz="0 0 ${cart_sz / 2}" parent="world" child="cart" />
+    <xacro:f_joint name="joint_cart" xyz="0 0 ${cart_sz / 2}" parent="base_link" child="cart" />
     <!-- joint_back_base is right_J8 -->
     <xacro:a_joint name="joint_back" type="revolute" xyz="${(cart_sx - back_base_sx) / 2} 0 ${cart_sz / 2}" parent="cart" child="back" axis="0 0 1" low="-1.58824" up="1.58824" />
