Commit message: add margin to bottom of sholder

File: src/melodic/myrobot_description/urdf/myrobot_v2.urdf.xacro (robot description, xacro)
@@ -64,6 +64,9 @@
     <xacro:property name="back_sy" value="0.144" />
     <xacro:property name="back_sz" value="0.86" />
+    <xacro:property name="sholder_base_sx" value="0.215" />
+    <xacro:property name="sholder_base_sy" value="0.02" />
+    <xacro:property name="sholder_base_sz" value="0.215" />
     <xacro:property name="sholder_sx" value="0.215" />
-    <xacro:property name="sholder_sy" value="0.215" />
+    <xacro:property name="sholder_sy" value="${0.215 + sholder_base_sy}" />
     <xacro:property name="sholder_sz" value="0.215" />
     <!-- //////////////////////////////////////////////////////////////////////////////////////////////////////////////////////////////////////////////////////////////// -->
@@ -96,11 +99,11 @@
     <xacro:d435 prefix="body" parent="body" xyz="${body_sx + 0.1} 0 0.1" rpy="0 ${radians(45)} 0" publish_pointcloud="1" />
     <!-- right arm -->
-    <xacro:sholder prefix="${prefix_1}" parent="body" xyz="${body_sx / 2 + body_spacer_length} -${body_sy / 2 + body_side_spacer_length} 0" l_xyz="0 0 -${sholder_sz / 2}" rpy="-${radians(90)} 0 0" size="${sholder_sx} ${sholder_sy} ${sholder_sz}" low="-0.01745" up="1.58824" />
-    <xacro:arm_with_soft_hand prefix="${prefix_1}" parent="${prefix_1}_sholder" xyz="${sholder_sx / 2} 0 -${sholder_sz / 2}" rpy="-${radians(90)} 0 -${radians(90)}" />
+    <xacro:sholder prefix="${prefix_1}" parent="body" xyz="${body_sx / 2 + body_spacer_length} -${body_sy / 2 + body_side_spacer_length} 0" l_xyz="0 0 -${sholder_sz / 2}" rpy="-${radians(90)} 0 0" size="${sholder_sx} ${sholder_sy} ${sholder_sz + 0.02}" low="-0.01745" up="1.58824" />
+    <xacro:arm_with_soft_hand prefix="${prefix_1}" parent="${prefix_1}_sholder" xyz="${sholder_sx / 2} 0 -${sholder_sz / 2 + 0.02}" rpy="-${radians(90)} 0 -${radians(90)}" />
     <!-- right camera -->
     <xacro:d435 prefix="${prefix_1}" parent="${prefix_1}_J6" xyz="0.1 0 0" rpy="0 ${radians(-90)} 0" publish_pointcloud="true" />
     <!-- left arm -->
-    <xacro:sholder prefix="${prefix_2}" parent="body" xyz="${body_sx / 2 + body_spacer_length} ${body_sy / 2 + body_side_spacer_length} 0" l_xyz="0 0 ${sholder_sy / 2}" rpy="-${radians(90)} 0 0" size="${sholder_sx} ${sholder_sy} ${sholder_sz}" low="-0.01745" up="1.58824" />
-    <xacro:arm_with_soft_hand prefix="${prefix_2}" parent="${prefix_2}_sholder" xyz="${sholder_sx / 2} 0 ${sholder_sz / 2}" rpy="-${radians(90)} 0 -${radians(90)}" />
+    <xacro:sholder prefix="${prefix_2}" parent="body" xyz="${body_sx / 2 + body_spacer_length} ${body_sy / 2 + body_side_spacer_length} 0" l_xyz="0 0 ${sholder_sy / 2}" rpy="-${radians(90)} 0 0" size="${sholder_sx} ${sholder_sy} ${sholder_sz + 0.02}" low="-0.01745" up="1.58824" />
+    <xacro:arm_with_soft_hand prefix="${prefix_2}" parent="${prefix_2}_sholder" xyz="${sholder_sx / 2} 0 ${sholder_sz / 2 + 0.02}" rpy="-${radians(90)} 0 -${radians(90)}" />
     <!-- left camera -->
     <xacro:d435 prefix="${prefix_2}" parent="${prefix_2}_J6" xyz="0.1 0 0" rpy="0 ${radians(-90)} 0" publish_pointcloud="true" />

Commit message: update sholder

File: src/melodic/myrobot_description/urdf/myrobot_v2.urdf.xacro (robot description, xacro)
@@ -13,8 +13,4 @@
     <xacro:include filename="$(find myrobot_description)/urdf/soft_hand/model.xacro" />
     <xacro:include filename="$(find myrobot_description)/urdf/utils.xacro" />
-    <xacro:macro name="sholder" params="prefix parent xyz l_xyz rpy size up low">
-        <xacro:a_joint name="${prefix}_joint_sholder" type="revolute" axis="0 0 1" parent="${parent}" child="${prefix}_sholder" xyz="${xyz}" rpy="${rpy}" up="${up}" low="${low}" />
-        <xacro:box_link name="${prefix}_sholder" xyz="${l_xyz}" size="${size}" color="red" />
-    </xacro:macro>
     <xacro:macro name="arm_with_soft_hand" params="prefix parent xyz rpy">
         <gazebo>
@@ -99,11 +95,19 @@
     <xacro:d435 prefix="body" parent="body" xyz="${body_sx + 0.1} 0 0.1" rpy="0 ${radians(45)} 0" publish_pointcloud="1" />
     <!-- right arm -->
-    <xacro:sholder prefix="${prefix_1}" parent="body" xyz="${body_sx / 2 + body_spacer_length} -${body_sy / 2 + body_side_spacer_length} 0" l_xyz="0 0 -${sholder_sz / 2}" rpy="-${radians(90)} 0 0" size="${sholder_sx} ${sholder_sy} ${sholder_sz + 0.02}" low="-0.01745" up="1.58824" />
-    <xacro:arm_with_soft_hand prefix="${prefix_1}" parent="${prefix_1}_sholder" xyz="${sholder_sx / 2} 0 -${sholder_sz / 2 + 0.02}" rpy="-${radians(90)} 0 -${radians(90)}" />
+    <xacro:a_joint name="${prefix_1}_joint_sholder" type="revolute" axis="0 0 1" parent="body" child="${prefix_1}_sholder" xyz="${body_sx / 2 + body_spacer_length} -${body_sy / 2 + body_side_spacer_length} 0" rpy="-${radians(90)} 0 0" low="-0.01745" up="1.58824" />
+    <link name="${prefix_1}_sholder">
+        <xacro:_box xyz="0 0 0" size="${sholder_sx} ${sholder_sy} 0.02" color="red" />
+        <xacro:_box xyz="${sholder_sx / 2 - 0.01} 0 -${sholder_sz / 2 + 0.01}" size="0.02 ${sholder_sy} ${sholder_sz}" color="red" />
+    </link>
+    <xacro:arm_with_soft_hand prefix="${prefix_1}" parent="${prefix_1}_sholder" xyz="${sholder_sx / 2} 0 -${sholder_sz / 2}" rpy="-${radians(90)} 0 -${radians(90)}" />
     <!-- right camera -->
     <xacro:d435 prefix="${prefix_1}" parent="${prefix_1}_J6" xyz="0.1 0 0" rpy="0 ${radians(-90)} 0" publish_pointcloud="true" />
     <!-- left arm -->
-    <xacro:sholder prefix="${prefix_2}" parent="body" xyz="${body_sx / 2 + body_spacer_length} ${body_sy / 2 + body_side_spacer_length} 0" l_xyz="0 0 ${sholder_sy / 2}" rpy="-${radians(90)} 0 0" size="${sholder_sx} ${sholder_sy} ${sholder_sz + 0.02}" low="-0.01745" up="1.58824" />
-    <xacro:arm_with_soft_hand prefix="${prefix_2}" parent="${prefix_2}_sholder" xyz="${sholder_sx / 2} 0 ${sholder_sz / 2 + 0.02}" rpy="-${radians(90)} 0 -${radians(90)}" />
+    <xacro:a_joint name="${prefix_2}_joint_sholder" type="revolute" axis="0 0 1" parent="body" child="${prefix_2}_sholder" xyz="${body_sx / 2 + body_spacer_length} ${body_sy / 2 + body_side_spacer_length} 0" rpy="-${radians(90)} 0 0" low="-0.01745" up="1.58824" />
+    <link name="${prefix_2}_sholder">
+        <xacro:_box xyz="0 0 0" size="${sholder_sx} ${sholder_sy} 0.02" color="red" />
+        <xacro:_box xyz="${sholder_sx / 2 - 0.01} 0 ${sholder_sz / 2 + 0.01}" size="0.02 ${sholder_sy} ${sholder_sz}" color="red" />
+    </link>
+    <xacro:arm_with_soft_hand prefix="${prefix_2}" parent="${prefix_2}_sholder" xyz="${sholder_sx / 2} 0 ${sholder_sz / 2}" rpy="-${radians(90)} 0 -${radians(90)}" />
     <!-- left camera -->
     <xacro:d435 prefix="${prefix_2}" parent="${prefix_2}_J6" xyz="0.1 0 0" rpy="0 ${radians(-90)} 0" publish_pointcloud="true" />

Commit message: update tip distance

File: src/melodic/myrobot_description/urdf/myrobot_v2.urdf.xacro (robot description, xacro)
@@ -26,6 +26,12 @@
         <xacro:vs087 prefix="${prefix}" />
         <xacro:soft_hand prefix="${prefix}" connected_to="${prefix}_J6" xyz="0 0 0" rpy="0 0 0" />
-        <xacro:f_joint name="${prefix}_joint_tip" xyz="0 0 0.105" parent="${prefix}_soft_hand_base_link" child="${prefix}_soft_hand_tip" />
-        <link name="${prefix}_soft_hand_tip" />
+        <xacro:f_joint name="${prefix}_joint_tip" xyz="0 0 0.3425" parent="${prefix}_soft_hand_base_link" child="${prefix}_soft_hand_tip" />
+        <link name="${prefix}_soft_hand_tip">
+            <visual>
+                <geometry>
+                    <box size="0.01 0.01 0.01" />
+                </geometry>
+            </visual>
+        </link>
     </xacro:macro>
     <xacro:macro name="d435" params="prefix parent xyz:='0 0 0' rpy='0 0 0' publish_pointcloud:=true">

Commit message: small fix

File: src/melodic/myrobot_description/urdf/myrobot_v2.urdf.xacro (robot description, xacro)
@@ -27,11 +27,5 @@
         <xacro:soft_hand prefix="${prefix}" connected_to="${prefix}_J6" xyz="0 0 0" rpy="0 0 0" />
         <xacro:f_joint name="${prefix}_joint_tip" xyz="0 0 0.3425" parent="${prefix}_soft_hand_base_link" child="${prefix}_soft_hand_tip" />
-        <link name="${prefix}_soft_hand_tip">
-            <visual>
-                <geometry>
-                    <box size="0.01 0.01 0.01" />
-                </geometry>
-            </visual>
-        </link>
+        <link name="${prefix}_soft_hand_tip" />
     </xacro:macro>
     <xacro:macro name="d435" params="prefix parent xyz:='0 0 0' rpy='0 0 0' publish_pointcloud:=true">

Commit message: update sholder position

File: src/melodic/myrobot_description/urdf/myrobot_v2.urdf.xacro (robot description, xacro)
@@ -60,9 +60,6 @@
     <xacro:property name="back_sy" value="0.144" />
     <xacro:property name="back_sz" value="0.86" />
-    <xacro:property name="sholder_base_sx" value="0.215" />
-    <xacro:property name="sholder_base_sy" value="0.02" />
-    <xacro:property name="sholder_base_sz" value="0.215" />
     <xacro:property name="sholder_sx" value="0.215" />
-    <xacro:property name="sholder_sy" value="${0.215 + sholder_base_sy}" />
+    <xacro:property name="sholder_sy" value="0.215" />
     <xacro:property name="sholder_sz" value="0.215" />
     <!-- //////////////////////////////////////////////////////////////////////////////////////////////////////////////////////////////////////////////////////////////// -->
@@ -70,5 +67,5 @@
     <!-- cart -->
     <link name="cart">
-        <xacro:_box size="${cart_sx} ${cart_sy} ${cart_sz}" />
+        <xacro:_box size="${cart_sx} ${cart_sy} ${cart_sz}" mass="100" />
         <xacro:_box size="${cart_box_sx} ${cart_box_sy} ${cart_box_sz}" xyz="-${(cart_sx - cart_box_sx) / 2} 0 ${(cart_sz + cart_box_sz) / 2}" />
     </link>
@@ -90,10 +87,10 @@
         <xacro:_cylinder xyz="${body_spacer_length / 2} 0 0" rpy="0 ${radians(90)} 0" radius="${body_spacer_radius}" length="${body_spacer_length}" color="green" />
         <xacro:_box xyz="${body_sx / 2 + body_spacer_length} 0 -${(body_sz) / 2 - body_spacer_radius}" size="${body_sx} ${body_sy} ${body_sz}" color="green" />
-        <xacro:_cylinder xyz="${body_sx / 2 + body_spacer_length} -${(body_sy + body_side_spacer_length) / 2} 0" rpy="${radians(90)} 0 0" radius="${body_side_spacer_radius}" length="${body_side_spacer_length}" color="green" />
-        <xacro:_cylinder xyz="${body_sx / 2 + body_spacer_length} ${(body_sy + body_side_spacer_length) /2} 0" rpy="${radians(90)} 0 0" radius="${body_side_spacer_radius}" length="${body_side_spacer_length}" color="green" />
+        <xacro:_cylinder xyz="${body_sx / 2 + body_spacer_length} -${(body_sy + body_side_spacer_length) / 2} -${(sholder_sz / 2) - body_side_spacer_radius}" rpy="${radians(90)} 0 0" radius="${body_side_spacer_radius}" length="${body_side_spacer_length}" color="green" />
+        <xacro:_cylinder xyz="${body_sx / 2 + body_spacer_length} ${(body_sy + body_side_spacer_length) /2} -${(sholder_sz / 2) - body_side_spacer_radius}" rpy="${radians(90)} 0 0" radius="${body_side_spacer_radius}" length="${body_side_spacer_length}" color="green" />
     </link>
     <xacro:d435 prefix="body" parent="body" xyz="${body_sx + 0.1} 0 0.1" rpy="0 ${radians(45)} 0" publish_pointcloud="1" />
     <!-- right arm -->
-    <xacro:a_joint name="${prefix_1}_joint_sholder" type="revolute" axis="0 0 1" parent="body" child="${prefix_1}_sholder" xyz="${body_sx / 2 + body_spacer_length} -${body_sy / 2 + body_side_spacer_length} 0" rpy="-${radians(90)} 0 0" low="-0.01745" up="1.58824" />
+    <xacro:a_joint name="${prefix_1}_joint_sholder" type="revolute" axis="0 0 1" parent="body" child="${prefix_1}_sholder" xyz="${body_sx / 2 + body_spacer_length} -${body_sy / 2 + body_side_spacer_length} -${(sholder_sz / 2) - body_side_spacer_radius}" rpy="-${radians(90)} 0 0" low="-0.01745" up="1.58824" />
     <link name="${prefix_1}_sholder">
         <xacro:_box xyz="0 0 0" size="${sholder_sx} ${sholder_sy} 0.02" color="red" />
@@ -104,5 +101,5 @@
     <xacro:d435 prefix="${prefix_1}" parent="${prefix_1}_J6" xyz="0.1 0 0" rpy="0 ${radians(-90)} 0" publish_pointcloud="true" />
     <!-- left arm -->
-    <xacro:a_joint name="${prefix_2}_joint_sholder" type="revolute" axis="0 0 1" parent="body" child="${prefix_2}_sholder" xyz="${body_sx / 2 + body_spacer_length} ${body_sy / 2 + body_side_spacer_length} 0" rpy="-${radians(90)} 0 0" low="-0.01745" up="1.58824" />
+    <xacro:a_joint name="${prefix_2}_joint_sholder" type="revolute" axis="0 0 1" parent="body" child="${prefix_2}_sholder" xyz="${body_sx / 2 + body_spacer_length} ${body_sy / 2 + body_side_spacer_length} -${(sholder_sz / 2) - body_side_spacer_radius}" rpy="-${radians(90)} 0 0" low="-0.01745" up="1.58824" />
     <link name="${prefix_2}_sholder">
         <xacro:_box xyz="0 0 0" size="${sholder_sx} ${sholder_sy} 0.02" color="red" />

Commit message: update model

File: src/melodic/myrobot_description/urdf/myrobot_v2.urdf.xacro (robot description, xacro)
@@ -40,4 +40,5 @@
     <xacro:property name="cart_sy" value="0.663" />
     <xacro:property name="cart_sz" value="0.294" />
+    <xacro:property name="cart_mass" value="100" />
     <xacro:property name="cart_box_sx" value="0.618" />
     <xacro:property name="cart_box_sy" value="0.663" />
@@ -64,8 +65,12 @@
     <link name="base_link" />
     <!-- cart -->
-    <link name="cart">
+    <link name="cart" mass="${cart_mass}">
         <xacro:_box size="${cart_sx} ${cart_sy} ${cart_sz}" mass="100" />
         <xacro:_box size="${cart_box_sx} ${cart_box_sy} ${cart_box_sz}" xyz="-${(cart_sx - cart_box_sx) / 2} 0 ${(cart_sz + cart_box_sz) / 2}" />
     </link>
+    <gazebo reference="cart">
+        <mu1>100.0</mu1>
+        <mu2>100.0</mu2>
+    </gazebo>
     <xacro:f_joint name="joint_cart" xyz="0 0 ${cart_sz / 2}" parent="base_link" child="cart" />
     <!-- joint_back_base is right_J8 -->

Commit message: remove unused plugin

File: src/melodic/myrobot_description/urdf/myrobot_v2.urdf.xacro (robot description, xacro)
@@ -13,13 +13,4 @@
     <xacro:include filename="$(find myrobot_description)/urdf/utils.xacro" />
     <xacro:macro name="arm_with_soft_hand" params="prefix parent xyz rpy">
-        <gazebo>
-            <!-- loading plugin: mimic joints works in gazebo now -->
-            <plugin name="gazebo_gripper_ros_control" filename="libroboticsgroup_gazebo_mimic_joint_plugin.so">
-                <joint>${prefix}_panda_finger_joint1</joint>
-                <mimicJoint>${prefix}_panda_finger_joint2</mimicJoint>
-                <multiplier>1.0</multiplier>
-                <offset>0.0</offset>
-            </plugin>
-        </gazebo>
         <xacro:f_joint name="${prefix}_joint_arm_base" xyz="${xyz}" rpy="${rpy}" parent="${parent}" child="${prefix}_base_link" />
         <xacro:vs087 prefix="${prefix}" />

Commit message: update model

File: src/melodic/myrobot_description/urdf/myrobot_v2.urdf.xacro (robot description, xacro)
@@ -56,6 +56,6 @@
     <link name="base_link" />
     <!-- cart -->
-    <link name="cart" mass="${cart_mass}">
-        <xacro:_box size="${cart_sx} ${cart_sy} ${cart_sz}" mass="100" />
+    <link name="cart">
+        <xacro:_box size="${cart_sx} ${cart_sy} ${cart_sz}" mass="${cart_mass}"/>
         <xacro:_box size="${cart_box_sx} ${cart_box_sy} ${cart_box_sz}" xyz="-${(cart_sx - cart_box_sx) / 2} 0 ${(cart_sz + cart_box_sz) / 2}" />
     </link>

Commit message: add world joint

File: src/melodic/myrobot_description/urdf/myrobot_v2.urdf.xacro (robot description, xacro)
@@ -54,4 +54,7 @@
     <xacro:property name="sholder_sz" value="0.215" />
     <!-- //////////////////////////////////////////////////////////////////////////////////////////////////////////////////////////////////////////////////////////////// -->
+    <!-- TODO: remove world_joint -->
+    <link name="world" />
+    <xacro:f_joint name="world_joint" parent="world" child="base_link" />
     <link name="base_link" />
     <!-- cart -->

Commit message: attachテストのための可動ジョイント追加

File: src/melodic/myrobot_description/urdf/myrobot_v2.urdf.xacro (robot description, xacro)
@@ -16,6 +16,20 @@
         <xacro:vs087 prefix="${prefix}" />
         <xacro:soft_hand prefix="${prefix}" connected_to="${prefix}_J6" xyz="0 0 0" rpy="0 0 0" />
+        <!-- virtual tip -->
         <xacro:f_joint name="${prefix}_joint_tip" xyz="0 0 0.3425" parent="${prefix}_soft_hand_base_link" child="${prefix}_soft_hand_tip" />
         <link name="${prefix}_soft_hand_tip" />
+        <!-- finger joints -->
+        <xacro:a_joint name="${prefix}_finger_1_joint" type="revolute" axis="1 0 0" parent="${prefix}_soft_hand_base_link" child="${prefix}_finger_1_link" xyz="0 0 0.3425"/>
+        <link name="${prefix}_finger_1_link">
+            <!-- ref: https://answers.ros.org/question/102276/this-robot-has-a-joint-named-foo-which-is-not-in-the-gazebo-model/ -->
+            <inertial>
+                <origin xyz="0 0 0" rpy="0 0 0" />
+                <mass value="0.001" />
+                <inertia
+                  ixx="0.001" ixy="0.0" ixz="0.0"
+                  iyy="0.001" iyz="0.0"
+                  izz="0.001" />
+            </inertial>
+        </link>
     </xacro:macro>
     <xacro:macro name="d435" params="prefix parent xyz:='0 0 0' rpy='0 0 0' publish_pointcloud:=true">
