Commit message: add hand joint

File: src/melodic/myrobot_description/urdf/myrobot_v2.urdf.xacro (robot description, xacro)
@@ -14,5 +14,9 @@
         <xacro:f_joint name="${prefix}_joint_arm_base" xyz="${arm_xyz}" rpy="${arm_rpy}" parent="${parent}" child="${prefix}_base_link" />
         <xacro:vs087 prefix="${prefix}" />
-        <xacro:soft_hand prefix="${prefix}" connected_to="${prefix}_J6" xyz="${hand_xyz}" rpy="${hand_rpy}" />
+        <xacro:f_joint name="${prefix}_joint_hand_joint" xyz="0 0 0" parent="${prefix}_J6" child="${prefix}_hand_joint" />
+        <link name="${prefix}_hand_joint">
+            <xacro:_cylinder xyz="0 0 0.02375" rpy="0 0 0" radius="0.0475" length="0.012" color="white" />
+        </link>
+        <xacro:soft_hand prefix="${prefix}" connected_to="${prefix}_hand_joint" xyz="${hand_xyz}" rpy="${hand_rpy}" />
         <!-- virtual tip -->
         <xacro:f_joint name="${prefix}_joint_tip" xyz="0 0 0.3425" parent="${prefix}_soft_hand_base_link" child="${prefix}_soft_hand_tip" />

Commit message: hand tipの軸修正

File: src/melodic/myrobot_description/urdf/myrobot_v2.urdf.xacro (robot description, xacro)
@@ -21,6 +21,6 @@
         <xacro:soft_hand prefix="${prefix}" connected_to="${prefix}_hand_joint" xyz="0 0 0" rpy="${hand_rpy}" />
         <!-- virtual tip -->
-        <xacro:f_joint name="${prefix}_joint_tip" xyz="0 0 0.3425" parent="${prefix}_soft_hand_base_link" child="${prefix}_soft_hand_tip" />
-        <link name="${prefix}_soft_hand_tip" />
+        <!-- <xacro:f_joint name="${prefix}_joint_tip" xyz="0 0 0.3425" parent="${prefix}_soft_hand_base_link" child="${prefix}_soft_hand_tip" />
+        <link name="${prefix}_soft_hand_tip" /> -->
         <!-- finger joints -->
         <xacro:a_joint name="${prefix}_finger_1_joint" type="revolute" axis="1 0 0" parent="${prefix}_soft_hand_base_link" child="${prefix}_finger_1_link" xyz="0 0 0.3425"/>
@@ -104,5 +104,6 @@
     <!-- TODO: デフォルト位置と可動範囲は要調節 -->
     <!-- joint_body is left_J8 (上下移動) -->
-    <xacro:a_joint name="joint_body" type="prismatic" xyz="-${back_base_sx - back_sx - back_spacer_radius} 0 ${back_spacer_length + back_base_sz + body_base_z_margin}" parent="back" child="body" axis="0 0 1" low="-0.001" up="0.495" />
+    <!-- <xacro:a_joint name="joint_body" type="prismatic" xyz="-${back_base_sx - back_sx - back_spacer_radius} 0 ${back_spacer_length + back_base_sz + body_base_z_margin}" parent="back" child="body" axis="0 0 1" low="-0.001" up="0.495" /> -->
+    <xacro:a_joint name="joint_body" type="prismatic" xyz="-${back_base_sx - back_sx - back_spacer_radius} 0 ${back_spacer_length + back_base_sz + body_base_z_margin}" parent="back" child="body" axis="0 0 1" low="0" up="0.495" />
     <link name="body">
         <xacro:_box xyz="${body_base_sx / 2} 0 ${body_base_sz / 2}" size="${body_base_sx} ${body_base_sy} ${body_base_sz}" color="green" />
@@ -116,5 +117,6 @@
     <xacro:d435 prefix="body" parent="body" xyz="${body_base_sx / 2 + 0.22} 0 ${body_base_sz + 0.015}" rpy="0 ${radians(45)} 0" publish_pointcloud="1" />
     <!-- right arm -->
-    <xacro:a_joint name="${prefix_1}_joint_sholder" type="revolute" axis="0 0 -1" parent="body" child="${prefix_1}_sholder" xyz="${body_sx / 2 + body_base_sx} -${body_sy / 2 + body_side_spacer_length} ${body_base_sz - body_side_spacer_radius - body_side_spacer_z_margin}" rpy="${radians(-90)} ${radians(90)} 0" low="-0.01745" up="1.58824" />
+    <!-- <xacro:a_joint name="${prefix_1}_joint_sholder" type="revolute" axis="0 0 -1" parent="body" child="${prefix_1}_sholder" xyz="${body_sx / 2 + body_base_sx} -${body_sy / 2 + body_side_spacer_length} ${body_base_sz - body_side_spacer_radius - body_side_spacer_z_margin}" rpy="${radians(-90)} ${radians(90)} 0" low="-0.01745" up="1.58824" /> -->
+    <xacro:a_joint name="${prefix_1}_joint_sholder" type="revolute" axis="0 0 -1" parent="body" child="${prefix_1}_sholder" xyz="${body_sx / 2 + body_base_sx} -${body_sy / 2 + body_side_spacer_length} ${body_base_sz - body_side_spacer_radius - body_side_spacer_z_margin}" rpy="${radians(-90)} ${radians(90)} 0" low="-0.01745" up="1.57079" />
     <link name="${prefix_1}_sholder">
         <xacro:_box xyz="0 0 -${0.02 / 2}" size="${sholder_sx} ${sholder_sy} 0.02" color="red" />
@@ -122,9 +124,12 @@
     </link>
     <xacro:arm_with_soft_hand prefix="${prefix_1}" parent="${prefix_1}_sholder" arm_xyz="${sholder_sx / 2} 0 -${sholder_sz / 2 + 0.02}" arm_rpy="${radians(-90)} 0 ${radians(-90)}" hand_rpy="0 0 ${radians(135)}" />
+    <xacro:f_joint name="${prefix_1}_joint_tip" xyz="0 0 0.3425" rpy="0 0 ${radians(-135)}" parent="${prefix_1}_soft_hand_base_link" child="${prefix_1}_soft_hand_tip" />
+    <link name="${prefix_1}_soft_hand_tip" />
     <!-- right camera -->
     <!-- <xacro:d435 prefix="${prefix_1}" parent="${prefix_1}_soft_hand_base_link" xyz="0 0 ${0.145 + 0.04}" rpy="${radians(45)} ${radians(-90)} 0" camera_xyz="0 0 -0.0125" publish_pointcloud="true" /> -->
     <xacro:d435 prefix="${prefix_1}" parent="${prefix_1}_hand_joint" xyz="0 0 0.012" rpy="0 0 0" camera_xyz="-0.0125 0 0.185" camera_rpy="0 ${radians(-90)} ${radians(180)}" publish_pointcloud="true" />
     <!-- left arm -->
-    <xacro:a_joint name="${prefix_2}_joint_sholder" type="revolute" axis="0 0 -1" parent="body" child="${prefix_2}_sholder" xyz="${body_sx / 2 + body_base_sx} ${body_sy / 2 + body_side_spacer_length} ${body_base_sz - body_side_spacer_radius - body_side_spacer_z_margin}" rpy="${radians(-90)} ${radians(90)} 0" low="-0.01745" up="1.58824" />
+    <!-- <xacro:a_joint name="${prefix_2}_joint_sholder" type="revolute" axis="0 0 -1" parent="body" child="${prefix_2}_sholder" xyz="${body_sx / 2 + body_base_sx} ${body_sy / 2 + body_side_spacer_length} ${body_base_sz - body_side_spacer_radius - body_side_spacer_z_margin}" rpy="${radians(-90)} ${radians(90)} 0" low="-0.01745" up="1.58824" /> -->
+    <xacro:a_joint name="${prefix_2}_joint_sholder" type="revolute" axis="0 0 -1" parent="body" child="${prefix_2}_sholder" xyz="${body_sx / 2 + body_base_sx} ${body_sy / 2 + body_side_spacer_length} ${body_base_sz - body_side_spacer_radius - body_side_spacer_z_margin}" rpy="${radians(-90)} ${radians(90)} 0" low="-0.01745" up="1.57079" />
     <link name="${prefix_2}_sholder">
         <xacro:_box xyz="0 0 ${0.02 /2}" size="${sholder_sx} ${sholder_sy} 0.02" color="red" />
@@ -132,4 +137,6 @@
     </link>
     <xacro:arm_with_soft_hand prefix="${prefix_2}" parent="${prefix_2}_sholder" arm_xyz="${sholder_sx / 2} 0 ${sholder_sz / 2 + 0.02}" arm_rpy="${radians(-90)} 0 ${radians(-90)}" hand_rpy="0 0 ${radians(-135)}" />
+    <xacro:f_joint name="${prefix_2}_joint_tip" xyz="0 0 0.3425" rpy="0 0 ${radians(135)}" parent="${prefix_2}_soft_hand_base_link" child="${prefix_2}_soft_hand_tip" />
+    <link name="${prefix_2}_soft_hand_tip" />
     <!-- left camera -->
     <!-- TODO: update camera direction (needs image flip) -->
