Commit message: reduce meshes

File: src/melodic/myrobot_description/urdf/soft_hand/model.xacro (robot description, xacro)
@@ -9,5 +9,5 @@
             <visual>
                 <geometry>
-                    <mesh filename="package://myrobot_description/urdf/soft_hand/0F_top_asm_soft_gripper_v1.stl" scale="0.001 0.001 0.001" />
+                    <mesh filename="package://myrobot_description/urdf/soft_hand/0F_top_asm_soft_gripper_v1_reduced.stl" scale="0.001 0.001 0.001" />
                 </geometry>
                 <origin xyz="0.0 0.0 0.138" rpy="${radians(90)} 0.0 0.0" />
@@ -18,5 +18,5 @@
             <collision>
                 <geometry>
-                    <mesh filename="package://myrobot_description/urdf/soft_hand/0F_top_asm_soft_gripper_v1.stl" scale="0.001 0.001 0.001" />
+                    <mesh filename="package://myrobot_description/urdf/soft_hand/0F_top_asm_soft_gripper_v1_reduced.stl" scale="0.001 0.001 0.001" />
                 </geometry>
             </collision>

Commit message: fix hand collision

File: src/melodic/myrobot_description/urdf/soft_hand/model.xacro (robot description, xacro)
@@ -20,4 +20,5 @@
                     <mesh filename="package://myrobot_description/urdf/soft_hand/0F_top_asm_soft_gripper_v1_reduced.stl" scale="0.001 0.001 0.001" />
                 </geometry>
+                <origin xyz="0.0 0.0 0.138" rpy="${radians(90)} 0.0 0.0" />
             </collision>
             <inertial>
